File: newTest/newTest.sch (KiCad schematic (older format))
At the start: 1 part

Commit message: 2nd commit
Parts:
- added R2: R, Resistor_SMD:R_0603_1608Metric_Pad1.05x0.95mm_HandSolder, symbol Device:R
- gave numbers to parts that had none: 1
Changed lines of the file:
@@
 $EndDescr
 $Comp
-L Device:R R?
+L Device:R R1
 U 1 1 60AD741E
 P 3675 2900
-F 0 "R?" V 3468 2900 50  0000 C CNN
+F 0 "R1" V 3468 2900 50  0000 C CNN
 F 1 "R" V 3559 2900 50  0000 C CNN
 F 2 "Resistor_SMD:R_0603_1608Metric_Pad1.05x0.95mm_HandSolder" V 3605 2900 50  0001 C CNN
@@
 	0    1    1    0
 $EndComp
+$Comp
+L Device:R R2
+U 1 1 60AD7907
+P 4875 2900
+F 0 "R2" V 4668 2900 50  0000 C CNN
+F 1 "R" V 4759 2900 50  0000 C CNN
+F 2 "Resistor_SMD:R_0603_1608Metric_Pad1.05x0.95mm_HandSolder" V 4805 2900 50  0001 C CNN
+F 3 "~" H 4875 2900 50  0001 C CNN
+	1    4875 2900
+	0    1    1    0
+$EndComp
